Commit message: UPDATE [2025.02.20] - marker detection: ArUco marker - CWS   . Main LiDAR: Warning/Stop zone definition     > Warning/Stop zone definition     > Detected obstacle message added   . Sub LiDAR:     > Warning/Stop zone definition     > Detected obstacle message added

File: urdf/ltrp.urdf (robot description, URDF)
Before this commit: robot ltrp, 14 links, 13 joints
Joints:
- joint JOINT_BASE: origin xyz=0.0 0.0 0.0 rpy=0.0 0.0 0.0 -> xyz=0.0 0.0 0.17 rpy=0.0 0.0 0.0
- joint JOINT_CASTER_LEFT: origin xyz=0.4 0.25 0.0762 rpy=0.4 0.0 0.0 -> xyz=0.4 0.25 -0.0938 rpy=0.4 0.0 0.0
- joint JOINT_CASTER_RIGHT: origin xyz=0.4 -0.25 0.0762 rpy=0.0 0.0 0.0 -> xyz=0.4 -0.25 -0.0938 rpy=0.0 0.0 0.0
- joint JOINT_CENTRAL_CAMERA: origin xyz=0.2 0.0 0.95 rpy=0.0 0.392699 0.0 -> xyz=0.2 0.0 0.83 rpy=0.0 0.392699 0.0
- joint JOINT_LEFT_CAMERA: origin xyz=0.1 0.2 0.95 rpy=0.0 0.392699 1.570796 -> xyz=0.1 0.2 0.83 rpy=0.0 0.392699 1.570796
- joint JOINT_LIDAR_MAIN: origin xyz=0.15 0.0 0.85 rpy=0.0 0.0 3.141592 -> xyz=0.15 0.0 0.68 rpy=0.0 0.0 0.0
- joint JOINT_RANGE_SENSOR_LEFT: origin xyz=0.15 0.25 0.8 rpy=0.0 0.52359866 1.570796 -> xyz=0.15 0.25 0.58 rpy=0.0 0.52359866 1.570796
- joint JOINT_RANGE_SENSOR_RIGHT: origin xyz=0.15 -0.25 0.8 rpy=0.0 0.52359866 -1.570796 -> xyz=0.15 -0.25 0.58 rpy=0.0 0.52359866 -1.570796
- joint JOINT_RIGHT_CAMERA: origin xyz=0.1 -0.2 0.95 rpy=0.0 0.392699 -1.570796 -> xyz=0.1 -0.2 0.83 rpy=0.0 0.392699 -1.570796
- joint JOINT_SUB_LIDAR: origin xyz=0.25 0.0 1.0 rpy=0.0 -0.785398 3.141592 -> xyz=0.15 0.0 0.58 rpy=0.0 -0.785398 3.141592
- joint JOINT_WHEEL_LEFT: origin xyz=0.0 0.3 0.1397 rpy=0.0 0.0 0.0 -> xyz=0.0 0.3 -0.0303 rpy=0.0 0.0 0.0
- joint JOINT_WHEEL_RIGHT: origin xyz=0.0 -0.3 0.1397 rpy=0.0 0.0 0.0 -> xyz=0.0 -0.3 -0.0303 rpy=0.0 0.0 0.0

Commit message: UPDATE & DEBUGGING [2025.03.11] - line detection - side camera orientation

File: urdf/ltrp.urdf (robot description, URDF)
Before this commit: robot ltrp, 14 links, 13 joints
Joints:
- joint JOINT_LEFT_CAMERA: origin xyz=0.1 0.2 0.83 rpy=0.0 0.392699 1.570796 -> xyz=0.1 0.2 0.83 rpy=0.0 0.0 0.523987
- joint JOINT_RIGHT_CAMERA: origin xyz=0.1 -0.2 0.83 rpy=0.0 0.392699 -1.570796 -> xyz=0.1 -0.2 0.83 rpy=0.0 0.0 -0.523987
